Commit message: REALNAV 2.9: SLAM, Teleop ve Full Rehber Güncellemesi

File: src/my_robot_description/urdf/my_robot.ros2_control.xacro (robot description, xacro)
@@ -2,26 +2,19 @@
 <robot xmlns:xacro="http://www.ros.org/wiki/xacro">
   <!--
-  ROS2 Control tanımı
-  NOT: Hardware interface kullanmıyoruz, serial bridge /joint_states yayınlıyor.
-  Controller'ın çalışması için minimal ros2_control tanımı gerekli.
+  ROS2 Control tanımı — MOCK (Sahte) Hardware
+  ============================================
+  Serial port iletişimini nav2_motor_bridge.py yapıyor.
+  Bu dosya sadece robot_state_publisher'ın URDF'yi kabul etmesi ve
+  controller yapısının tanımlı olması için gerekli.
+  ÖNEMLİ: my_robot_hardware/DiffDriveSystem KULLANILMIYOR!
+  O plugin /dev/ttyAMA0'ı açmaya çalışıyor ve nav2_motor_bridge ile
+  çakışarak encoder verisi kaybolmasına neden oluyordu.
   -->
   <xacro:macro name="my_robot_ros2_control" params="name prefix">
     <ros2_control name="${name}" type="system">
       <hardware>
-        <!--
-        Hardware interface yok, serial bridge kullanıyoruz.
-        Controller /joint_states topic'ini kullanacak.
-        Bu sadece controller'ın başlaması için gerekli.
-        fake_components/GenericSystem kullanıyoruz (ros2_control paketinde var).
-        -->
-        <plugin>my_robot_hardware/DiffDriveSystem</plugin>
-        <param name="port">/dev/ttyAMA0</param>
-        <param name="baud">115200</param>
-        <param name="ticks_per_rev">4000</param>
-        <param name="max_wheel_rad_s">20.0</param>
-        <param name="min_pwm">30</param>
-        <param name="cmd_deadband_rad_s">0.05</param>
+        <plugin>mock_components/GenericSystem</plugin>
+        <param name="fake_sensor_commands">false</param>
         <param name="state_following_offset">0.0</param>
-        <param name="fake_sensor_commands">false</param>
       </hardware>
       <joint name="${prefix}left_wheel_joint">

File: src/my_robot_description/urdf/my_robot.urdf.xacro (robot description, xacro)
@@ -16,9 +16,9 @@
   <!-- Robot ölçüleri (Gerçek robot ölçüleri) -->
   <xacro:property name="PI" value="3.1415926535897931"/>
-  <xacro:property name="base_width" value="0.55" />
+  <xacro:property name="base_width" value="0.43" />
   <xacro:property name="base_length" value="0.60" />
   <xacro:property name="base_height" value="0.24" />
   <xacro:property name="wheel_len" value="0.030" />
-  <xacro:property name="wheel_radius" value="0.055" />
+  <xacro:property name="wheel_radius" value="0.050" />
   <xacro:property name="caster_wheel_radius" value="0.055" />
   <xacro:property name="axle_offset" value="0.10" />
